File: FlightControllerPCB/MCU.kicad_sch (KiCad schematic)
At the start: 11 parts, among them SW3 SW_Push, SW4 SW_SPDT, U5 STM32F745VGTx

Commit message: Sanity check+Error fixes
Parts:
- added J5: I2C/SPI Header, symbol Connector:Conn_01x08_Pin
- added J6: Timer Header, symbol Connector:Conn_01x06_Pin
- added R15, R22: 4.7k, symbol Device:R
- added R16, R17, R18: 100, symbol Device:R
- added R19, R2, R20, R21: 10k, symbol Device:R
Connections:
- net +3.3V: now also J5.1 (Pin_1), J6.2 (Pin_2), R15.1, R2.1, R22.1
- net GND: now also J5.8 (Pin_8), J6.6 (Pin_6), R19.1, R20.1, R21.1
- net at U5.1 (PE2): now also J5.2 (Pin_2)
- net Gen GPIO/ SPI MOSI: now reaches U5.17 (PC2)
- net Gen GPIO/ SPI MOSI: now also J5.7 (Pin_7)
- net at U5.2 (PE3): now also J5.3 (Pin_3)
- net at U5.3 (PE4): now also J5.4 (Pin_4), R2.2
- net at U5.4 (PE5): now also R16.2
- net at U5.5 (PE6): now also R17.2
- net at U5.58 (PD11): now also J5.5 (Pin_5), R15.2
- net at U5.59 (PD12): now also J5.6 (Pin_6), R22.2
- net at U5.60 (PD13): now also R18.2
- net RC_TX: now reaches U5.63 (PC6)
- net RC_RX: now reaches U5.64 (PC7)
- new net: J6.5 (Pin_5), R18.1, R21.2
- new net: J6.4 (Pin_4), R17.1, R20.2
- new net: J6.3 (Pin_3), R16.1, R19.2
- new net +5V: J6.1 (Pin_1)
- no-connect marks 0 -> 55
Other:
- note removed: "- Jeson connector (UART+JST) - USB(D+,D-) - 6 pin micro JST for GPS - extra header + resistors"
- note removed: "- RC conn"

Commit message: XT30 conn
Other:
- note added: "+ extra solder pads"
- note added: "ESC conn"
Changed lines of the file:
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@@
 	(generator_version "10.0")
 	(paper "A4")
+	(text "+ extra solder pads\n"
+		(exclude_from_sim no)
+		(at 42.164 108.712 0)
+		(effects
+			(font
+				(size 1.27 1.27)
+			)
+		)
+	)
+	(text "ESC conn"
+		(exclude_from_sim no)
+		(at 239.268 69.85 0)
+		(effects
+			(font
+				(size 1.27 1.27)
+			)
+		)
+	)
+	(text "+ extra solder pads\n"
+		(exclude_from_sim no)
+		(at 41.402 80.01 0)
+		(effects
+			(font
+				(size 1.27 1.27)
+			)
+		)
+	)
 	(junction
 		(at 73.66 27.94)
