File: FlightControllerPCB/power.kicad_sch (KiCad schematic)
At the start: 10 parts, among them J4 USB_C_Receptacle_USB2.0_16P, U13 D3V3XA4B10LP, U16 AMS1117-3.3

Commit message: actually the IMU+baro changes
Parts:
- added C5: 1uF, symbol Device:C
- added U2: AP2112K-1.8, Package_TO_SOT_SMD:SOT-23-5, symbol Regulator_Linear:AP2112K-1.8
Connections:
- net +3.3V: now also C5.1, U2.1 (VIN), U2.3 (EN)
- net GND: now also C5.2, U2.2 (GND)
- new net +1.8V: U2.5 (VOUT)

Commit message: Power circuit
Other:
- moved on the sheet: C13, C16, C5, D2, D3, J4, R9, U13, U16, U2

Commit message: early MCU setup
Parts:
- added C17, C18: 10uF, symbol Device:C
- added C19: 220pF, symbol Device:C
- added C20: .1uF, symbol Device:C
- added C21, C22: 22uF, symbol Device:C
- added D1: SS34, Diode_SMD:D_SMA, symbol Diode:SS34
- added IC1: MP1584EN-LF-Z, MP1584EN-LF-Z:SOIC127P600X170-9N, symbol MP1584EN-LF-Z:MP1584EN-LF-Z
- added L1: 8.2uH, symbol Device:L
- added R11, R12, R3: 100k, symbol Device:R
- added R13: 43.2k, symbol Device:R
- added R14: 8.2k, symbol Device:R
Connections:
- net +5V: now also C21.1, C22.1, L1.2, R13.2
- net GND: now also C17.2, C18.2, C21.2, C22.2, D1.2 (A), IC1.5 (GND), IC1.9 (EP), R11.1, R12.1, R14.2
- net Data+ renamed USB Data +
- net Data- renamed USB Data -
- new net: C19.1, IC1.3 (COMP)
- new net: C19.2, R12.2
- new net: C20.2, D1.1 (K), IC1.1 (SW), L1.1
- new net: IC1.2 (EN), R3.1
- new net: IC1.4 (FB), R13.1, R14.1
- new net: IC1.6 (FREQ), R11.2
- new net: C20.1, IC1.8 (BST)
- new net +24V: C17.1, C18.1, IC1.7 (VIN), R3.2
Other:
- note added: "Sanity check all circuits"
- moved on the sheet: C13, C16, C5, D2, D3, J4, R9, U13, U16, U2

Commit message: Sanity check+Error fixes
Parts:
- added C24: 1uF, symbol Device:C
- added C25: .1uF, symbol Device:C
- R9: value 1K -> 470
Connections:
- net +1.8V: now also C24.1
- net +3.3V: now also C25.1
- net GND: now also C24.2, C25.2
Other:
- note removed: "Sanity check all circuits"
- moved on the sheet: C16, D2, D3, J4, R9, U13

Commit message: XT30 conn
Parts:
- added BT1: 6S Lipo, symbol Device:Battery
- added J7: XT30, symbol Connector_Generic:Conn_01x02
Connections:
- net +24V: now also BT1.1 (+), J7.2 (Pin_2)
- net GND: now also BT1.2 (-), J7.1 (Pin_1)
